File: open offline weather station.kicad_sch (KiCad schematic)
At the start: 7 parts

Commit message: Add files via upload
just a small tweak to some names in the schematic
Parts:
- renumbered 2004A1 to 2004A, DHT1 to DHT11, HC-SR1 to HC-SR04, MQ-1 to MQ-2, ds1 to ds3231
Other:
- added sheet Battery Protection (weather station.kicad_sch)
- added sheet Powersupply (weather station.kicad_sch)
- added sheet Remote sensor (weather station.kicad_sch)
- title: (none) -> open offline weather station
